Commit message: updated

File: src/test_slam/urdf/rawbot.gazebo.xacro (robot description, xacro)
@@ -25,6 +25,6 @@
     </plugin>
   </gazebo>
-  <!-- camera -->
-  <gazebo reference="camera">
+  <!-- camera_link -->
+  <gazebo reference="camera_link">
     <sensor type="depth" name="camera1">
         <always_on>1</always_on>
@@ -48,5 +48,5 @@
             <alwaysOn>true</alwaysOn>
             <updateRate>10.0</updateRate>
-            <cameraName>camera</cameraName>
+            <cameraName>camera_link</cameraName>
             <frameName>camera_link_optical</frameName>
             <imageTopicName>/rawbot/camera/rgb/image_raw</imageTopicName>
@@ -73,5 +73,5 @@
     <sensor type="ray" name="head_hokuyo_sensor">
       <pose>0 0 0 0 0 0</pose>
-      <visualize>false</visualize>
+      <visualize>true</visualize>
       <update_rate>40</update_rate>
       <ray>
@@ -80,6 +80,8 @@
             <samples>720</samples>
             <resolution>1</resolution>
-            <min_angle>-1.570796</min_angle>
-            <max_angle>1.570796</max_angle>
+            <!-- <min_angle>-1.570796</min_angle>
+            <max_angle>1.570796</max_angle> -->
+            <min_angle>-2.655</min_angle>
+            <max_angle>2.655</max_angle>
           </horizontal>
         </scan>
@@ -105,3 +107,16 @@
     </sensor>
   </gazebo>
+  <!-- since there are multiple uvc and uvc_support link, we include their gazebo color in their corresponding macro -->
+  <gazebo reference="wheel_left_link">
+    <material>Gazebo/Black</material>
+  </gazebo>
+  <gazebo reference="wheel_right_link">
+    <material>Gazebo/Black</material>
+  </gazebo>
+  <gazebo reference="base_link">
+    <material>Gazebo/Red</material>
+  </gazebo>
+  <gazebo reference="camera_link">
+    <material>Gazebo/Orange</material>
+  </gazebo>
 </robot>

File: src/test_slam/urdf/rawbot.urdf.xacro (robot description, xacro)
@@ -4,4 +4,5 @@
     <xacro:include filename="$(find test_slam)/urdf/common_properties.xacro"/>
     <xacro:include filename="$(find test_slam)/urdf/uvc.macro.xacro"/>
+    <xacro:include filename="$(find test_slam)/urdf/sonar.macro.xacro"/>
     <link name="base_footprint"/>
     <joint name="base_joint" type="fixed">
@@ -21,5 +22,5 @@
                 izz="0.1" />
         </inertial>
-        <collision name='collision'>
+        <collision>
             <origin xyz="0 0 0" rpy=" 0 0 0"/>
             <geometry>
@@ -34,5 +35,5 @@
             <material name="red"/>
         </visual>
-        <collision name='back_caster_collision'>
+        <collision>
             <origin xyz="-0.15 0 -0.05" rpy=" 0 0 0"/>
             <geometry>
@@ -40,5 +41,5 @@
             </geometry>
         </collision>
-        <visual name='back_caster_visual'>
+        <visual> <!--back_caster_visual-->
             <origin xyz="-0.15 0 -0.05" rpy=" 0 0 0"/>
             <geometry>
@@ -47,5 +48,5 @@
             <material name="green"/><!--Doesn't work here-->
         </visual>
-        <collision name='front_caster_collision'>
+        <collision>
             <origin xyz="0.15 0 -0.05" rpy=" 0 0 0"/>
             <geometry>
@@ -53,5 +54,5 @@
             </geometry>
         </collision>
-        <visual name='front_caster_visual'>
+        <visual><!--front_caster_visual-->
             <origin xyz="0.15 0 -0.05" rpy=" 0 0 0"/>
             <geometry>
@@ -62,10 +63,10 @@
     </link>
     <!--uvc-->
-    <xacro:uvc_support_link name="uvc_support_link1" origin_xyz="0 0 0.075"/>
-    <xacro:uvc_link name="uvc_link1" origin_xyz="0.05 0 0.6"/>
-    <xacro:uvc_link name="uvc_link2" origin_xyz="0 0.05 0.6"/>
-    <xacro:uvc_link name="uvc_link3" origin_xyz="-0.05 0 0.6"/>
-    <xacro:uvc_link name="uvc_link4" origin_xyz="0 -0.05 0.6"/>
-    <xacro:uvc_support_link name="uvc_support_link2" origin_xyz="0 0 1.125"/>
+    <xacro:cuboid name="uvc_support1" origin_xyz="0 0 0.075" box_size=".15 .15 .05"/>
+    <xacro:uvc_link name="uvc1" origin_xyz="0.05 0 0.6"/>
+    <xacro:uvc_link name="uvc2" origin_xyz="0 0.05 0.6"/>
+    <xacro:uvc_link name="uvc3" origin_xyz="-0.05 0 0.6"/>
+    <xacro:uvc_link name="uvc4" origin_xyz="0 -0.05 0.6"/>
+    <xacro:cuboid name="uvc_support2" origin_xyz="0 0 1.125" box_size=".15 .15 .05"/>
     <!--wheel_left_link-->
     <link name="wheel_left_link">
@@ -79,5 +80,5 @@
             />
         </inertial>
-        <collision name='left_wheel_collision'>
+        <collision>
             <origin xyz="0 0 0" rpy=" 0 1.5707 1.5707"/>
             <geometry>
@@ -85,5 +86,5 @@
             </geometry>
         </collision>
-        <visual name='left_wheel_visual'>
+        <visual>
             <origin xyz="0 0 0" rpy=" 0 1.5707 1.5707"/>
             <geometry>
@@ -111,5 +112,5 @@
                 izz="0.1"/>
         </inertial>
-        <visual name='right_wheel_visual'>
+        <visual>
             <origin xyz="0 0 0" rpy="0 1.5707 1.5707"/>
             <geometry>
@@ -118,5 +119,5 @@
             <material name="dark"/>
         </visual>
-        <collision name='right_wheel_collision'>
+        <collision>
             <origin xyz="0 0 0" rpy="0 1.5707 1.5707" />
             <geometry>
@@ -133,6 +134,6 @@
         <dynamics damping="1.0" friction="1.0"/>
     </joint>
-    <!--camera-->
-    <link name="camera">
+    <!--camera_link-->
+    <link name="camera_link">
         <inertial>
             <mass value="0.1"/>
@@ -143,5 +144,5 @@
                 izz="1e-6"/>
         </inertial>
-        <visual name='camera_visual'>
+        <visual>
             <origin xyz="0 0 0" rpy="0 0 0"/>
             <geometry>
@@ -150,5 +151,5 @@
             <material name="orange"/>
         </visual>
-        <collision name='camera_collision'>
+        <collision>
             <origin xyz="0 0 0" rpy="0 0 0" />
             <geometry>
@@ -158,6 +159,6 @@
     </link>
     <joint name="camera_joint" type="fixed" >
-        <origin xyz="0.2 0 0" rpy="0 0 0"/>
-        <child link="camera"/>
+        <origin xyz="0.2 0 0.075" rpy="0 0 0"/>
+        <child link="camera_link"/>
         <parent link="base_link"/>
         <axis xyz="0 1 0" rpy="0 0 0"/>
@@ -165,9 +166,10 @@
     <joint name="camera_optical_joint" type="fixed">
         <origin xyz="0 0 0" rpy="-1.5707 0 -1.5707"/>
-        <parent link="camera"/>
+        <parent link="camera_link"/>
         <child link="camera_link_optical"/>
     </joint>
     <link name="camera_link_optical"/>
     <!--LIDAR-->
+    <xacro:cuboid name="lidar_support" origin_xyz="0.15 0 0.075" box_size=".05 .05 .05"/>
     <link name="base_scan">
         <inertial>
@@ -189,17 +191,23 @@
             <origin xyz="0 0 0" rpy="0 0 0" />
             <geometry>
-                <box size="0.1 0.1 0.1"/>
+                <box size="0.05 0.05 0.05"/>
             </geometry>
         </collision>
     </link>
     <joint type="fixed" name="scan_joint">
-        <origin xyz="0.15 0 0.075" rpy="0 0 0"/>
+        <origin xyz="0.15 0 0.125" rpy="0 0 0"/>
         <child link="base_scan"/>
         <parent link="base_link"/>
         <axis xyz="0 1 0" rpy="0 0 0"/>
     </joint>
-    <!--Doesn't work here-->
-    <gazebo reference="wheel_left_link">
-        <material>Gazebo/Green</material>
+    <!-- SONAR -->
+    <xacro:sonar name="fl_sonar" origin_xyz="0.2 0.1 0.0" origin_rpy="0 0 0"/>
+    <xacro:sonar name="fc_sonar" origin_xyz="0.2 0.0 0.0" origin_rpy="0 0 0"/>
+    <xacro:sonar name="fr_sonar" origin_xyz="0.2 -0.1 0.0" origin_rpy="0 0 0"/>
+    <xacro:sonar name="bl_sonar" origin_xyz="-0.2 0.1 0.0" origin_rpy="0 0 3.14"/>
+    <xacro:sonar name="bc_sonar" origin_xyz="-0.2 0.0 0.0" origin_rpy="0 0 3.14"/>
+    <xacro:sonar name="br_sonar" origin_xyz="-0.2 -0.1 0.0" origin_rpy="0 0 3.14"/>
+    <gazebo reference="camera_link">
+        <material>Gazebo/Orange</material>
     </gazebo>
 </robot>

File: src/test_slam/urdf/uvc.macro.xacro (robot description, xacro)
@@ -2,5 +2,5 @@
 <robot xmlns:xacro="http://www.ros.org/wiki/xacro">
     <!-- <xacro:include filename="$(find test_slam)/urdf/common_properties.xacro"/> -->
-    <xacro:macro name="uvc_support_link" params="name origin_xyz">
+    <xacro:macro name="cuboid" params="name origin_xyz box_size">
         <!--uvc_support-->
         <link name="${name}_link">
@@ -16,5 +16,5 @@
                 <origin xyz="0.0 0 0" rpy=" 0 0 0"/>
                 <geometry>
-                    <box size=".15 .15 .05"/>
+                    <box size="${box_size}"/>
                 </geometry>
             </collision>
@@ -22,5 +22,5 @@
                 <origin xyz="0.0 0 0" rpy=" 0 0 0"/>
                 <geometry>
-                    <box size=".15 .15 .05"/>
+                    <box size="${box_size}"/>
                 </geometry>
                 <material name="white"/>
@@ -32,4 +32,7 @@
             <child link="${name}_link" />
         </joint>
+        <gazebo reference="${name}_link">
+            <material>Gazebo/Green</material>
+        </gazebo>
     </xacro:macro>
     <xacro:macro name="uvc_link" params="name origin_xyz" >
@@ -63,4 +66,7 @@
             <child link="${name}_link" />
         </joint>
+        <gazebo reference="${name}_link">
+            <material>Gazebo/Blue</material>
+        </gazebo>
     </xacro:macro>
 </robot>
