Commit message: updated

File: src/test_slam/urdf/sonar.macro.xacro (robot description, xacro)
@@ -37,5 +37,5 @@
             <sensor type="ray" name="${name}">
                 <pose>0 0 0 0 0 0</pose>
-                <visualize>true</visualize>
+                <visualize>true</visualize> <!--For visualization-->>
                 <update_rate>5</update_rate>
                 <ray>
@@ -56,5 +56,5 @@
                     <range>
                         <min>0.02</min>
-                        <max>4</max>
+                        <max>1</max> <!--changed form 4 to 1 for resolving obstacle issue -->
                         <resolution>0.01</resolution>
                     </range>

File: src/trial_mob_rob_description/urdf/trial_mob_rob.xacro (robot description, xacro)
@@ -4,4 +4,10 @@
 <xacro:include filename="$(find trial_mob_rob_description)/urdf/trial_mob_rob.trans" />
 <xacro:include filename="$(find trial_mob_rob_description)/urdf/trial_mob_rob.gazebo" />
+<!-- <link name="base_footprint"/>
+<joint name="base_joint" type="fixed">
+    <origin xyz="0 0 0.1" rpy="0 0 0" />
+    <parent link="base_footprint"/>
+    <child link="base_link" />
+</joint> -->
 <link name="base_link">
   <inertial>
